File: JugendHackt-Badge-Display.kicad_sch (KiCad schematic)
At the start: 140 parts, among them J1 USB_C_Receptacle_USB2.0, J2 Conn_01x30_Female, J3 Conn_01x02, Q1 S8050, Q2 S8050, SW1 K1-1506SN-01, SW2 SW_Push, SW3 SW_Push, SW4 SW_SPDT, U1 RM-V8xxC_TR1, U2 SRV05-4, U3 CH340C, U4 ESP32-WROOM-32, U5 SDB628, U6 TLV62568DBV, U7 MCP73831-2-OT

Commit message: feat: Final PCB
Parts:
- D10: renamed from D13; LCSC (none) -> C965557
- D11: renamed from D9; LCSC (none) -> C965557
- D12: renamed from D8; LCSC (none) -> C965557
- D7: renamed from D11; LCSC (none) -> C965557
- D8: renamed from D12; LCSC (none) -> C965557
- D9: renamed from D7; LCSC (none) -> C965557
- IO1, IO12, TP3: now left out of the parts list
- IO10: renamed from IO8; now left out of the parts list
- IO11: renamed from IO10; now left out of the parts list
- IO2: renamed from IO3; now left out of the parts list
- IO3: renamed from IO5; now left out of the parts list
- IO4: renamed from IO7; now left out of the parts list
- IO5: renamed from IO9; now left out of the parts list
- IO6: renamed from IO11; now left out of the parts list
- IO7: renamed from IO2; now left out of the parts list
- IO8: renamed from IO4; now left out of the parts list
- IO9: renamed from IO6; now left out of the parts list
- J1: renamed from J3; footprint Connector_Molex:Molex_PicoBlade_53261-0271_1x02-1MP_P1.25mm_Horizontal -> Connector_JST:JST_PH_S2B-PH-SM4-TB_1x02-1MP_P2.00mm_Horizontal; LCSC (none) -> C442222
- J3: renamed from J1; LCSC (none) -> C2874568
- TP1: renamed from TP6; now left out of the parts list
- TP10: renamed from TP40; now left out of the parts list
- TP12: renamed from TP4; now left out of the parts list
- TP13: renamed from TP5; now left out of the parts list
- TP14: renamed from TP7; now left out of the parts list
- TP15: renamed from TP9; now left out of the parts list
- TP16: renamed from TP10; now left out of the parts list
- TP17: renamed from TP11; now left out of the parts list
- TP18: renamed from TP12; now left out of the parts list
- TP19: renamed from TP13; now left out of the parts list
- TP2: renamed from TP8; now left out of the parts list
- TP20: renamed from TP14; now left out of the parts list
- TP21: renamed from TP15; now left out of the parts list
- TP22: renamed from TP16; now left out of the parts list
- TP23: renamed from TP17; now left out of the parts list
- TP24: renamed from TP19; now left out of the parts list
- TP25: renamed from TP21; now left out of the parts list
- TP26: renamed from TP23; now left out of the parts list
- TP27: renamed from TP25; now left out of the parts list
- TP28: renamed from TP27; now left out of the parts list
- TP29: renamed from TP30; now left out of the parts list
- TP30: renamed from TP31; now left out of the parts list
- TP31: renamed from TP32; now left out of the parts list
- TP32: renamed from TP33; now left out of the parts list
- TP33: renamed from TP34; now left out of the parts list
- TP34: renamed from TP35; now left out of the parts list
- TP35: renamed from TP36; now left out of the parts list
- TP4: renamed from TP18; now left out of the parts list
- TP5: renamed from TP20; now left out of the parts list
- TP6: renamed from TP22; now left out of the parts list
- TP7: renamed from TP24; now left out of the parts list
- TP8: renamed from TP26; now left out of the parts list
- TP9: renamed from TP29; now left out of the parts list
- U2: renamed from U4; LCSC (none) -> C701343
- renumbered C22 to C1, C24 to C10, C25 to C11, C8 to C12, C4 to C13, C5 to C14, C19 to C15, C10 to C16, C12 to C17, C6 to C18, C7 to C19, C1 to C2, C18 to C22, C9 to C23, C14 to C24, C13 to C25, C11 to C26, C16 to C27, C15 to C28, C2 to C4, C17 to C5, C23 to C6, C27 to C7, C29 to C8, C28 to C9, D4 to D1, D1 to D4, D6 to D5, D5 to D6, R22 to R1, R24 to R10, R5 to R11, R2 to R12, R3 to R13, R4 to R14, R20 to R15, R19 to R16, R30 to R17, R8 to R18, R28 to R19, R25 to R2, R7 to R20, R1 to R21, R6 to R22, R11 to R23, R21 to R24, R23 to R25, R9 to R26, R26 to R27, R27 to R28, R10 to R29, R13 to R3, R12 to R4, R14 to R5, R17 to R6, R18 to R7, R16 to R8, R15 to R9, SW4 to SW2, SW2 to SW4, TP41 to TP11, TP38 to TP36, TP39 to TP38, TP28 to TP39, U6 to U1, U2 to U3, U3 to U4, U7 to U6, U1 to U7
Connections:
- net GND: now also J1.1 (Pin_1); no longer J1.2 (Pin_2)
- net at F1.2: now also J1.2 (Pin_2); no longer J1.1 (Pin_1)
Other:
- moved on the sheet: J1, TP10
